Commit message: add sonar

File: src/zx_description/urdf/W2A/imu.xacro (robot description, xacro)
@@ -2,12 +2,42 @@
 <robot xmlns:xacro="http://www.ros.org/wiki/xacro" name="imu">
     <xacro:macro name="imu" params="prefix:=imu">
+        <!-- IMU的link -->
+        <link name="${prefix}_link">
+            <visual>
+                <origin xyz="0 0 0" rpy="0 0 0" />
+                <geometry>
+                    <!-- 这里假设IMU为一个简单的立方体 -->
+                    <box size="0.001 0.001 0.001" />
+                </geometry>
+                <material name="gray">
+                    <color rgba="0.5 0.5 0.5 1.0" />
+                    <!-- 灰色 -->
+                </material>
+            </visual>
+            <collision>
+                <origin xyz="0 0 0" rpy="0 0 0" />
+                <geometry>
+                    <box size="0.001 0.001 0.001" />
+                </geometry>
+            </collision>
+            <inertial>
+                <mass value="0.01" />
+                <!-- 假设质量为0.01kg -->
+                <inertia ixx="0.001" ixy="0" ixz="0" iyy="0.001" iyz="0" izz="0.001" />
+            </inertial>
+        </link>
+        <!-- IMU与父节点的连接joint，这里为固定连接 -->
+        <joint name="${prefix}_joint" type="fixed">
+            <parent link="base_link" />
+            <child link="${prefix}_link" />
+            <origin xyz="0 0 0.05" rpy="0 0 0" />
+        </joint>
         <gazebo reference="${prefix}_link">
             <sensor type="imu" name="imu_sensor">
                 <always_on>true</always_on>
-                <update_rate>100</update_rate>
+                <update_rate>50.0</update_rate>
                 <visualize>true</visualize>
-                <topic>__default_topic__</topic>
                 <plugin name="imu_plugin" filename="libgazebo_ros_imu_sensor.so">
-                    <topicName>/imu</topicName>
+                    <topicName>imu/data</topicName>
                     <frameName>imu_link</frameName>
                     <updateRateHZ>100.0</updateRateHZ>
@@ -17,5 +47,4 @@
                     <initialOrientationAsReference>false</initialOrientationAsReference>
                 </plugin>
-                <pose>0 0 0 0 0 0</pose>
             </sensor>
         </gazebo>

File: src/zx_description/urdf/W2A/sonar.xacro (robot description, xacro)
@@ -4,5 +4,5 @@
   <xacro:property name="sonar_radius" value="0.001" />
   <xacro:property name="sonar_height" value="0.001" />
-  <xacro:macro name="add_sonar" params="pos xyz rpy">
+  <xacro:macro name="sonar" params="pos xyz rpy">
     <link name="${pos}_sonar">
       <visual>

File: src/zx_description/urdf/W2A/w2a.xacro (robot description, xacro)
@@ -3,8 +3,10 @@
 	xmlns:xacro="http://www.ros.org/wiki/xacro">
 	<xacro:include filename="$(find zx_description)/urdf/W2A/w2a.urdf" />
-	<xacro:include filename="$(find zx_description)/urdf/W2A/rplidar.xacro" />
 	<xacro:include filename="$(find zx_description)/urdf/W2A/differential_drive_controller.xacro" />
 	<xacro:include filename="$(find zx_description)/urdf/W2A/arm_controller.xacro" />
-	<xacro:rplidar prefix="laser"/>
+	<xacro:include filename="$(find zx_description)/urdf/W2A/rplidar.xacro" />
+	<xacro:include filename="$(find zx_description)/urdf/W2A/imu.xacro" />
+	<xacro:include filename="$(find zx_description)/urdf/W2A/depth_camera.xacro" />
+	<xacro:include filename="$(find zx_description)/urdf/W2A/sonar.xacro" />
 	<xacro:differential_drive_controller/>
 	<xacro:transmission_block joint_name="joint_1"/>
@@ -15,3 +17,9 @@
 	<xacro:transmission_block joint_name="claw_joint_1"/>
 	<xacro:transmission_block joint_name="claw_joint_2"/>
+	<xacro:rplidar prefix="laser"/>
+	<xacro:imu prefix="imu"/>
+	<xacro:depth_camera prefix="camera"/>
+	<xacro:sonar pos="front" xyz=" 0.182 0 0.03" rpy="0 0 0"/>
+    <xacro:sonar pos="left" xyz=" 0.0 0.14 0.03" rpy="0 0 0.78"/>
+    <xacro:sonar pos="right" xyz=" 0.0 -0.14 0.03" rpy="0 0 -0.78"/>
 </robot>
